Commit message: corrected urdf param

File: urdf/kobuki_carto.urdf (robot description, URDF)
Before this commit: robot kobuki_standalone, 10 links, 9 joints
Joints:
- joint base_joint: origin xyz=0 0 0 rpy=0 0 0 -> xyz=0 0 0.01 rpy=0 0 0

File: urdf/kobuki_gazebo_carto.urdf (robot description, URDF)
Before this commit: robot kobuki_standalone, 10 links, 9 joints
Joints:
- joint base_joint: origin xyz=0 0 0 rpy=0 0 0 -> xyz=0 0 0.1 rpy=0 0 0

Commit message: add office maps

File: urdf/kobuki_carto.urdf (robot description, URDF)
Before this commit: robot kobuki_standalone, 10 links, 9 joints
Joints:
- joint base_joint: origin xyz=0 0 0.01 rpy=0 0 0 -> xyz=0 0 0.0102 rpy=0 0 0
